File: single_quad_rt_hp/hardware/motor_controller/logic_regulator.kicad_sch (KiCad schematic)
At the start: 10 parts, among them IC401 LM2596SX-5.0_NOPB, IC402 NCP1117ST33T3G

Commit message: [single_quad_rt_hp] removing switching regs and simplifying the sceme
Parts:
- removed C403, C404: 68u, Capacitor_SMD:CP_Elec_6.3x7.7, symbol Device:C_Polarized_Small_US
- removed C405: 330u, Capacitor_SMD:CP_Elec_10x10, symbol Device:C_Polarized_Small_US
- removed D401: D_Schottky, Diode_SMD:D_SMC, symbol Device:D_Schottky
- removed IC401: LM2596SX-5.0_NOPB, KTT0005B, symbol SamacSys_Parts:LM2596SX-5.0_NOPB
- removed L401: 47u, Manual_Parts:YSPI1365-470M, symbol Device:L_Small
- removed TP401: TestPoint, TestPoint:TestPoint_Pad_1.5x1.5mm, symbol Connector:TestPoint
Connections:
- net SWITCH_OUT_5V renamed VBUS_IN
- no-connect marks 2 -> 1
Other:
- note added: "Stage 1: Linear Regulator"
- note removed: "* Used WBENCH Tools to calculate passive components * LM2596SX-5.0/NOPB 15V-20V to 5.00V @ 2.5A"
- note removed: "150 kHz (58.35 mV p-p) --> 5V @ 2.5"
- note removed: "550mV 5A"
- note removed: "DCR: 57.5 mOhm"
- note removed: "ESR: 35mOhm"
- note removed: "ESR: 90 mOhm"
- note removed: "Specification V_{IN} = 12V V_{OUT} = 3.3V @ 1A 2 Stages: - 12V -> 5V (Switching) - 5V -> 3.3V (Linear)"
- note removed: "Stage 1: Switching Regulator"
- note removed: "Stage 2: Linear Regulator"
- note removed: "This stage may not be necessary anymore"
- moved on the sheet: C401, C402, IC402
