File: single_quad_rt_hp/hardware/motor_controller/motor_controller.kicad_pcb (KiCad board)
At the start: 4 copper layers, 94.4 x 70.1 mm, 66 parts, among them IC301 LM5085MY_NOPB, IC401 LM2596SX-5.0_NOPB, IC402 NCP1117ST33T3G, IC601 N25S830HAT22I, J201 Robot Power Bus, J501 Motor Driver (Control), J502 Motor Driver (Power), J503 Motor Connector, J601 Show Control Interface, J602 Limit Switch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

Commit message: [single_quad_rt_hp] removing switching regs and simplifying the sceme
Parts:
- removed C101: 4.7u, Capacitor_SMD:C_0603_1608Metric
- removed C102, C103, C104, C105: 100n, Capacitor_SMD:C_0402_1005Metric
- removed C106, C302: 1u, Capacitor_SMD:C_0603_1608Metric
- removed C107: 10n, Capacitor_SMD:C_0402_1005Metric
- removed C108, C109: 27p, Capacitor_SMD:C_0603_1608Metric
- removed C301: 1n, Capacitor_SMD:C_0805_2012Metric
- removed C303: 82u, Capacitor_SMD:CP_Elec_8x11.9
- removed C304: 6.8n, Capacitor_SMD:C_0805_2012Metric
- removed C305: 56u, Capacitor_SMD:CP_Elec_6.3x5.8
- removed C401, C402: 10u, Capacitor_SMD:C_0603_1608Metric
- removed C403, C404: 68u, Capacitor_SMD:CP_Elec_6.3x7.7
- removed C405: 330u, Capacitor_SMD:CP_Elec_10x10
- removed C501: 470u, Capacitor_THT:CP_Radial_D8.0mm_P3.50mm
- removed C601: 100n, Resistor_SMD:R_0402_1005Metric
- removed D101: BLUE, LED_SMD:LED_0603_1608Metric
- removed D201, D202: GREEN, LED_SMD:LED_0603_1608Metric
- removed D301, D401: D_Schottky, Diode_SMD:D_SMC
- removed D601, D602, D603, D604, D605: D_TVS, SamacSys_Parts:SOD2512X110N
- removed IC301: LM5085MY_NOPB, SamacSys_Parts:SOP65P490X109-9N
- removed IC401: LM2596SX-5.0_NOPB, SamacSys_Parts:KTT0005B
- removed IC402: NCP1117ST33T3G, SamacSys_Parts:SOT230P700X180-4N
- removed IC601: N25S830HAT22I, SamacSys_Parts:SOP65P640X120-8N
- removed J201: Robot Power Bus, Connector_PinSocket_2.54mm:PinSocket_1x02_P2.54mm_Vertical
- removed J501: Motor Driver (Control), Connector_PinSocket_2.54mm:PinSocket_1x08_P2.54mm_Vertical
- removed J502: Motor Driver (Power), Connector_PinSocket_2.54mm:PinSocket_1x08_P2.54mm_Vertical
- removed J503: Motor Connector, Connector_PinHeader_2.54mm:PinHeader_1x06_P2.54mm_Vertical
- removed J601: Show Control Interface, Connector_PinSocket_2.54mm:PinSocket_1x04_P2.54mm_Vertical
- removed J602: Limit Switch, Connector_PinSocket_2.54mm:PinSocket_1x03_P2.54mm_Vertical
- removed J603: SWD Connector, Connector_PinHeader_2.54mm:PinHeader_2x04_P2.54mm_Vertical
- removed L301: 6.8u, Manual_Parts:YSPIA1770-6R8M
- removed L401: 47u, Manual_Parts:YSPI1365-470M
- removed MOSFET301: SI7149DP-T1-GE3, SamacSys_Parts:SI7149DP-T1-GE3
- removed R101: 10k, Resistor_SMD:R_0603_1608Metric
- removed R102, R201, R202: 1.5k, Resistor_SMD:R_0603_1608Metric
- removed R103: 36, Resistor_SMD:R_0402_1005Metric
- removed R301: 2.55k, Resistor_SMD:R_0402_1005Metric
- removed R302: 10m, Resistor_SMD:R_1210_3225Metric
- removed R303: 205k, Resistor_SMD:R_0402_1005Metric
- removed R304: 10k, Resistor_SMD:R_0402_1005Metric
- removed R305: 1.15k, Resistor_SMD:R_0402_1005Metric
- removed R601, R602, R603, R604: 49.9, Resistor_SMD:R_0402_1005Metric
- removed TP101, TP201, TP202, TP203, TP401: TestPoint, TestPoint:TestPoint_Pad_1.5x1.5mm
- removed U101: STM32F302C8Tx, Package_QFP:LQFP-48_7x7mm_P0.5mm
- removed Y101: 16MHz, SamacSys_Parts:ABM816000MHZB2T
Routing:
- net +3V3: track 238.3 -> 0.00 mm, vias 9 -> 0
- net +12V: track 73.1 -> 0.00 mm
- net ENC_A: track 65.4 -> 0.00 mm, vias 2 -> 0
- net ENC_B: track 60.7 -> 0.00 mm, vias 2 -> 0
- net GND: track 44.5 -> 0.00 mm, vias 568 -> 0
- net PWR_MOTOR_P: track 34.8 -> 0.00 mm
- net PWR_MOTOR_N: track 32.6 -> 0.00 mm
- net /(5) Motor Driver/VM: track 28.3 -> 0.00 mm
- net SW_LIMIT: track 24.2 -> 0.00 mm
- net ACTUATOR_POWER_FLAG: track 22.9 -> 0.00 mm
- net CAN_TX: track 20.2 -> 0.00 mm
- net SYS_JTMS-SWDIO: track 19.7 -> 0.00 mm
- net NRST: track 19.4 -> 0.00 mm, vias 2 -> 0
- net CAN_RX: track 19.3 -> 0.00 mm
- net I2C_SDA: track 18.5 -> 0.00 mm
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- removed copper zone on F.Cu, net +12V
- removed copper zone on F.Cu, net +3V3
- removed copper zone on F.Cu, net /(2) Power Supply/(3) Actuator Regulator/ISEN
- removed copper zone on F.Cu, net /(2) Power Supply/(3) Actuator Regulator/MOSFETT_OUT
- removed copper zone on F.Cu, net /(2) Power Supply/(4) Logic Regulator/OUTPUT_SW
- removed copper zone on F.Cu, net /(2) Power Supply/POWER_BUS
- removed copper zone on F.Cu, net GND
- removed copper zone on In1.Cu, net GND
- removed copper zone on In2.Cu, net GND
- removed copper zone on F.Cu, net PWR_MOTOR_N
- removed copper zone on F.Cu, net PWR_MOTOR_P
- removed copper zone on F.Cu, net SWITCH_OUT_5V
Other:
- board outline removed
- board text removed: "(+)"
- board text removed: "+"
- board text removed: "12V @ 6A 349.38 kHz"
- board text removed: "16 MHz"
- board text removed: "5V @ 2.5A 150 kHz"
- board text removed: "ACTUATOR REGULATION"
- board text removed: "B1 (HULA) v0.2 Alexander Adranly 12/22"
- board text removed: "CAN_RX"
- board text removed: "CAN_TX"
- board text removed: "CROSS-RIPPLE TP [15V - 20V]"
- board text removed: "ENC_A"
- board text removed: "ENC_B"
- board text removed: "I2C_SCL"
- board text removed: "I2C_SDA"
- board text removed: "LOGIC REGULATION"
- board text removed: "MOTOR (-)"
- board text removed: "MOTOR CONNTECTOR"
- board text removed: "MOTOR DRIVER - CONTROL INTERFACE"
- board text removed: "MOTOR DRIVER - OUTPUT"
- board text removed: "MOTOR(+)"
- board text removed: "N25S830HAT22I"
- board text removed: "NOTE: Do not run at high currents without CAP installed >>>>"
- board text removed: "NRST"
- board text removed: "POWER BUS [15V - 20V @ 6A]"
- board text removed: "SERIAL WIRE DEBUGGER"
- board text removed: "SWCLK"
- board text removed: "SWDIO"
- board text removed: "SWO"
- board text removed: "SW_LIMIT"
- board text removed: "pololu 18v17"
